File: electronics/power.sch.kicad_sch (KiCad schematic)
At the start: 6 parts, among them U1 MCP73831-2-OT

Commit message: Part number for battery charge controller
Parts:
- U1: LCSC Part # (none) -> C424093
Changed lines of the file:
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@@
+			)
+		)
+		(property "LCSC Part #" "C424093"
+			(at 52.07 38.1 0)
+			(hide yes)
+			(show_name no)
+			(do_not_autoplace no)
+			(effects
+				(font
+					(size 1.27 1.27)
+				)
 			)
 		)

Commit message: Initial power design, excepting solenoid supply
Parts:
- added C11: .1uF, symbol Device:C_Small
- added C5, C7: 4.7uF, symbol Device:C
- added C8: 1.8uF, symbol Device:C_Small
- added D2: B5817W, Diode_SMD:D_SOD-123, symbol Device:D_Schottky
- added L1: 2.2uH, Inductor_SMD:L_Coilcraft_LPS3010, symbol Device:L
- added Q2: MDD2301, Package_TO_SOT_SMD:SOT-23, symbol Transistor_FET:Q_PMOS_GSD
- added R3: 1.2Meg, symbol Device:R_Small
- added R4: 220k, symbol Device:R_Small
- added R5: 100R, symbol Device:R_Small
- added R6: 10k, symbol Device:R
- added U3: TLV74311, Package_TO_SOT_SMD:SOT-23-5, symbol irrigation-controller:TLV74311PDVBR
- added U4: TPS63000, Package_SON:Texas_DRC0010J_ThermalVias, symbol Regulator_Switching:TPS63000
Connections:
- net +BATT: now also Q2.3 (D)
- net GND: now also C11.2, C5.2, C7.2, R4.2, R6.1, U3.2 (GND), U4.11 (PGND), U4.3 (PGND), U4.9 (GND)
- net VBUS: now also D2.2 (A), Q2.1 (G), R6.2
- new net: D2.1 (K), Q2.2 (S), R5.1, U4.5 (VIN)
- new net: C11.1, R5.2, U4.6 (EN), U4.7 (PS/SYNC), U4.8 (VINA)
- new net: L1.1, U4.2 (L2)
- new net: L1.2, U4.4 (L1)
- new net: C8.2, R3.2, R4.1, U4.10 (FB)
- new net +1V1: C7.1, U3.5 (OUT)
- new net +3V3: C5.1, C8.1, R3.1, U3.1 (IN), U3.3 (EN), U4.1 (VOUT)
Other:
- note added: "1.1V regulator for RP2354 (I love the RP series but the bespoke parts are getting out of hand)"
- note added: "3.3V Buck/Boost regulator"
- note added: "Battery Charge Controller"
- note added: "Check that USB spec will not exceed 7V"

Commit message: Microcontroller design
Other:
- moved on the sheet: C11, C8, D2, L1, Q2, R3, R4, R5, R6, U4
