File: electronics/water-controller.kicad_sch (KiCad schematic)
At the start: 12 parts, among them J1 USB_C_Receptacle_USB2.0_16P, SW2 RST, U2 STM32L432KBUx, Y1 32.768kHz

Commit message: Battery charge controller
Other:
- added sheet Battery Controller and Regulator (power.sch.kicad_sch)
Changed lines of the file:
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@@
+		)
+	)
+	(sheet
+		(at 185.42 124.46)
+		(size 81.28 35.56)
+		(exclude_from_sim no)
+		(in_bom yes)
+		(on_board yes)
+		(dnp no)
+		(fields_autoplaced yes)
+		(stroke
+			(width 0.1524)
+			(type solid)
+		)
+		(fill
+			(color 0 0 0 0)
+		)
+		(property "Sheetname" "Battery Controller and Regulator"
+			(at 185.42 123.7484 0)
+			(show_name no)
+			(do_not_autoplace no)
+			(effects
+				(font
+					(size 1.27 1.27)
+				)
+				(justify left bottom)
+			)
+		)
+		(property "Sheetfile" "power.sch.kicad_sch"
+			(at 185.42 160.6046 0)
+			(show_name no)
+			(do_not_autoplace no)
+			(effects
+				(font
+					(size 1.27 1.27)
+				)
+				(justify left top)
+			)
+		)
+		(instances
+			(project "water-controller"
+				(path "/90ee257d-08bc-4d08-b044-1d51d5c028cf"
+					(page "2")
+				)
+			)
 		)
 	)

Commit message: Initial power design, excepting solenoid supply
Parts:
- removed U2: STM32L432KBUx, Package_DFN_QFN:QFN-32-1EP_5x5mm_P0.5mm_EP3.45x3.45mm, symbol MCU_ST_STM32L4:STM32L432KBUx
- added U2: RP2354A, Package_DFN_QFN:QFN-60-1EP_7x7mm_P0.4mm_EP3.4x3.4mm, symbol MCU_RaspberryPi:RP2354A
Connections:
- net GND: now also J1.SH (SHIELD); no longer J1.S1 (SHIELD)
- new net: U2.1 (IOVDD), U2.11 (IOVDD), U2.20 (IOVDD), U2.30 (IOVDD), U2.38 (IOVDD), U2.45 (IOVDD)
- new net: U2.23 (DVDD), U2.39 (DVDD), U2.6 (DVDD)
- no-connect marks 2 -> 7

Commit message: Microcontroller design
Parts:
- added C12, C13, C14, C15, C16, C17, C18, C19, C20, C21: .1uF, symbol Device:C
- added C22, C23: 15pF, Capacitor_SMD:C_0603_1608Metric, symbol Device:C
- added R13, R15: 27, Resistor_SMD:R_0603_1608Metric, symbol Device:R
- added R16: 5.1k, Resistor_SMD:R_0402_1005Metric, symbol Device:R
- added R7: 1k, symbol Device:R
- added R8: 1k, Resistor_SMD:R_0402_1005Metric, symbol Device:R
- added SW3, SW4: BOOT, cat:TS-1088-AR02016, symbol Switch:SW_Push
- added TP1: SWCLK, symbol Connector:TestPoint
- added TP2: SWDIO, symbol Connector:TestPoint
- added Y2: 12MHz, Crystal:Crystal_SMD_Abracon_ABM8G-4Pin_3.2x2.5mm, symbol Device:Crystal_GND24
- C1: value 0.1uF -> 4.7uF; footprint Capacitor_SMD:C_0402_1005Metric -> (none); LCSC Part # C1525 -> (none)
- C3: value 4.7uF -> .1uF
- C6: value 0.1uF -> .1uF; footprint Capacitor_SMD:C_0402_1005Metric -> (none); LCSC Part # C1525 -> (none)
Connections:
- net +3V3: now also U2.1 (IOVDD), U2.11 (IOVDD), U2.20 (IOVDD), U2.30 (IOVDD), U2.38 (IOVDD), U2.44 (ADC_AVDD), U2.45 (IOVDD), U2.46 (VREG_AVDD), U2.49 (VREG_VIN), U2.53 (USB_OTP_VDD), U2.54 (QSPI_IOVDD), C13.1, C14.1, C15.1, C16.1, C17.1, C18.1, C19.1, C20.1, C21.1, R16.2; no longer C3.1, C6.1
- net GND: now also U2.47 (VREG_PGND), U2.50 (VREG_FB), U2.61 (GND), C12.2, C13.2, C14.2, C15.2, C16.2, C17.2, C18.2, C19.2, C20.2, C21.2, C22.1, C23.1, SW3.2, SW4.2, Y2.2, Y2.4
- net USB_D+: now also R15.2
- net USB_D-: now also R13.2
- net at U2.21 (XIN): now also C22.2, Y2.3
- net at U2.22 (XOUT): now also R8.2
- net +1V1: now reaches U2.23 (DVDD), U2.39 (DVDD), U2.6 (DVDD)
- net +1V1: now also C3.1, C6.1, C12.1
- net at U2.24 (SWCLK): now also TP2.1
- net at U2.25 (SWDIO): now also TP1.1
- net RUN: now reaches U2.26 (RUN)
- net RUN: now also R16.1, SW4.1
- net at U2.51 (USB_DM): now also R13.1
- net at U2.52 (USB_DP): now also R15.1
- net at U2.60 (~{QSPI_SS}): now also R7.2
- new net: C23.2, R8.1, Y2.1
- new net ~{USB_BOOT}: R7.1, SW3.1
- no-connect marks 7 -> 8
Other:
- note added: "-"
- note added: "Decoupling caps for RP2354"
- note added: "Decoupling caps for RP2354 DVDD"
- note added: "Irrigation Controller Mainboard"
- note added: "Pins 53/54 share a 100nF cap"
- note added: "Planning to keep 12MHz oscillator on at all times and just eat the power hit External low frequency clocks are expensive and the internal oscillator is way too imprecise"
- note added: "Shut down internal regulator in software to save ~400uA"
- note added: "for vreg_vin"

Commit message: Solenoid driver
Other:
- added sheet Solenoid Drivers (drivers.kicad_sch)
Changed lines of the file:
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@@
+		)
+	)
+	(sheet
+		(at 227.33 99.06)
+		(size 39.37 21.59)
+		(exclude_from_sim no)
+		(in_bom yes)
+		(on_board yes)
+		(dnp no)
+		(fields_autoplaced yes)
+		(stroke
+			(width 0.1524)
+			(type solid)
+		)
+		(fill
+			(color 0 0 0 0)
+		)
+		(property "Sheetname" "Solenoid Drivers"
+			(at 227.33 98.3484 0)
+			(show_name no)
+			(do_not_autoplace no)
+			(effects
+				(font
+					(size 1.27 1.27)
+				)
+				(justify left bottom)
+			)
+		)
+		(property "Sheetfile" "drivers.kicad_sch"
+			(at 227.33 121.2346 0)
+			(show_name no)
+			(do_not_autoplace no)
+			(effects
+				(font
+					(size 1.27 1.27)
+				)
+				(justify left top)
+			)
+		)
+		(instances
+			(project "water-controller"
+				(path "/90ee257d-08bc-4d08-b044-1d51d5c028cf"
+					(page "3")
+				)
+			)
 		)
 	)
